File: eagle/rev_b/cpu_eval_board.sch (EAGLE design)
At the start: 42 parts, among them Y1 8MHz

Commit message: cpu eval board wip
Parts:
- removed L1: (no value), microbuilder:INDUCTOR_0603
- added C20, C21: 10uF X7R 0805, microbuilder:CAP_CERAMIC_0805
- added C22, C23: 0.1uF, microbuilder:CAP_CERAMIC0603
- added FB1: (no value), microbuilder:FERRITE_0805
- added LED3: (no value), microbuilder:LED0603
- added R13, R17: 2.2K, microbuilder:RESISTOR0603
- added R3: 680, microbuilder:RESISTOR0603
- added R4: 0, microbuilder:RESISTOR0603
- added U$25: MIC37100, keves:MIC37100
- added U1: 24LC512, microbuilder:EEPROM_I2C_SOIC8_GENERIC
Connections:
- net PA0 renamed SW_USER
- net PA11 renamed USB_DM
- net PA12 renamed USB_DP
- net PD12 renamed LED1
- net PD13 renamed LED2
- new net N$7: C23.P$1, R13.2, R17.2, R4.1, U1.VCC
- new net N$8: LED3.A, R3.1
- new net SCL: R17.1, STM32F407XX1.PB10, U1.SCL
- new net SDA: R13.1, STM32F407XX1.PB11, U1.SDA
- net 3.3V: now also C21.P$1, C22.P$1, R3.2, R4.2, U$25.VO; no longer L1.1
- net 5.0V: now also C20.P$2, U$25.VI
- net GND: now also C20.P$1, C21.P$2, C22.P$2, C23.P$2, LED3.C, U$25.GND, U$25.GND_TAB, U1.A0, U1.A1, U1.A2, U1.GND, U1.WP
- net N$4: now also FB1.P$2; no longer L1.2
Other:
- moved on the sheet: JTAG

Commit message: cpu eval board wip
Parts:
- added C24: 100nF, microbuilder:CAP_CERAMIC0603
- added CONN_LCD: (no value), con-harting-ml:ML16
- added IC5: 74HC595D, 74xx-eu:74HC595D
- added JP2: (no value), microbuilder:JUMPER3
- added LCD_POT1, LCD_POT2: 10K 67WR10KLF, BaseApp:TRIMPOT-67W
- added Q1: BC337, transistor-small-signal:BC337
- added R18: 10K, microbuilder:RESISTOR_0603
- added R19, R20, R21, R22: 1K, microbuilder:RESISTOR_0603
Connections:
- new net LCD_B-: CONN_LCD.15, Q1.B, R18.1
- new net LCD_D0: CONN_LCD.8, IC5A.QA
- new net LCD_D1: CONN_LCD.7, IC5A.QB
- new net LCD_D2: CONN_LCD.10, IC5A.QC
- new net LCD_D3: CONN_LCD.9, IC5A.QD
- new net LCD_D4: CONN_LCD.12, IC5A.QE
- new net LCD_D5: CONN_LCD.11, IC5A.QF
- new net LCD_D6: CONN_LCD.14, IC5A.QG
- new net LCD_D7: CONN_LCD.13, IC5A.QH, STM32F407XX1.PD7
- new net LCD_E1: CONN_LCD.5, R21.2, STM32F407XX1.PC8
- new net LCD_RS: CONN_LCD.3, IC5A.SER, R20.2, STM32F407XX1.PA8
- new net LCD_RW: CONN_LCD.6, IC5A.G, R22.2, STM32F407XX1.PC11
- new net LCD_SER_RCLK: IC5A.RCK, STM32F407XX1.PD3
- new net LCD_SER_SCLK: IC5A.SCK, STM32F407XX1.PD6
- new net LCD_V0: CONN_LCD.4, LCD_POT1.S
- new net LCD_VD: C24.P$2, CONN_LCD.1, IC5A.SCL, IC5P.VCC, JP2.2, LCD_POT1.E, R20.1, R21.1, R22.1
- new net N$19: Q1.C, R19.1
- new net N$20: LCD_POT2.S, R19.2
- net 3.3V: now also FB1.P$1, JP2.3
- net 5.0V: now also CONN_LCD.16, JP2.1, LCD_POT2.A, R18.2
- net GND: now also C24.P$1, CONN_LCD.2, IC5P.GND, LCD_POT1.A, LCD_POT2.E, Q1.E

Commit message: wip
Parts:
- removed CONN_LCD: (no value), con-harting-ml:ML16
- added C25: 0.1uF/500v, microbuilder:CAP_CERAMIC0603
- added C26, C27: 18pF, microbuilder:CAP_CERAMIC0603
- added D1, D2: 1N4148WS, microbuilder:DIODESOD-323
- added H1, H2, H3, H4: MOUNT-HOLE3.3, holes:MOUNT-HOLE3.3
- added IC1, IC2: 6N138S-TA1, 6n138:6N138SMD
- added LCD1: NHD-C0220AA-FSW-FTW, NHD-C0220AA-FSW-FTW:NHD-C0220AA-FSW-FTW
- added MIDI_IN1, MIDI_IN2, MIDI_OUT1, MIDI_OUT2: MIDIJACK, keves:MIDIJACK
- added R23: 1M, microbuilder:RESISTOR0603
- added R24, R25, R26, R29, R30, R31: 220, microbuilder:RESISTOR_0603
- added R27, R32: 4.7K, microbuilder:RESISTOR_0603
- added R28, R33: 1K, microbuilder:RESISTOR_0603
- added R34, R35, R36, R37, R38: 10K, microbuilder:RESISTOR_0603
- added R39, R40, R41, R42, R43: POT, pot-alps:POT_US
- added S1, S2, S3, S4, S5: (no value), og-switch:40-XX
- added SW1, SW2: Encoder, switch-alps:EC12E_SW
Connections:
- new net A0: R39.S, STM32F407XX1.PC1
- new net A1: R40.S, STM32F407XX1.PC2
- new net A2: R41.S, STM32F407XX1.PA1
- new net A3: R42.S, STM32F407XX1.PA4
- new net A4: R43.S, STM32F407XX1.PC4
- new net MIDI_IN1: IC1.VO, R28.1, STM32F407XX1.PA3
- new net MIDI_IN2: IC2.VO, R33.1, STM32F407XX1.PD9
- new net MIDI_OUT1: R25.1, STM32F407XX1.PA2
- new net MIDI_OUT2: R30.1, STM32F407XX1.PD8
- new net N$21: C25.P$1, R23.2, U$14.S1, U$14.S2
- new net N$23: MIDI_OUT1.5, R25.2
- new net N$24: MIDI_OUT1.4, R26.2
- new net N$25: MIDI_IN1.4, R24.2
- new net N$26: D1.C, IC1.A, R24.1
- new net N$27: D1.A, IC1.C, MIDI_IN1.5
- new net N$28: IC1.VB, R27.1
- new net N$29: MIDI_OUT2.5, R30.2
- new net N$30: MIDI_OUT2.4, R31.2
- new net N$31: MIDI_IN2.4, R29.2
- new net N$32: D2.C, IC2.A, R29.1
- new net N$33: D2.A, IC2.C, MIDI_IN2.5
- new net N$34: IC2.VB, R32.1
- new net SCS_D0: STM32F407XX1.PE8, SW1G$1.B
- new net SCS_D1: STM32F407XX1.PE9, SW1G$1.A
- new net SCS_D10: STM32F407XX1.PC15, SW2G$2.2
- new net SCS_D2: STM32F407XX1.PE10, SW1G$2.2
- new net SCS_D3: R34.1, S1.P, S1.P1, STM32F407XX1.PE11
- new net SCS_D4: R35.1, S2.P, S2.P1, STM32F407XX1.PE12
- new net SCS_D5: R36.1, S3.P, S3.P1, STM32F407XX1.PE13
- new net SCS_D6: R37.1, S4.P, S4.P1, STM32F407XX1.PE14
- new net SCS_D7: R38.1, S5.P, S5.P1, STM32F407XX1.PE15
- new net SCS_D8: STM32F407XX1.PC13, SW2G$1.B
- new net SCS_D9: STM32F407XX1.PC14, SW2G$1.A
- net 3.3V: now also R34.2, R35.2, R36.2, R37.2, R38.2, R39.A, R40.A, R41.A, R42.A, R43.A
- net 5.0V: now also IC1.VCC, IC2.VCC, LCD1.A, R26.1, R28.2, R31.1, R33.2, STM32F407XX1.PA9; no longer CONN_LCD.16
- net GND: now also C25.P$2, C26.P$1, C27.P$1, IC1.GND, IC2.GND, LCD1.GND, MIDI_OUT1.2, MIDI_OUT2.2, R23.1, R27.2, R32.2, R39.E, R40.E, R41.E, R42.E, R43.E, S1.S, S1.S1, S2.S, S2.S1, S3.S, S3.S1, S4.S, S4.S1, S5.S, S5.S1, SW1G$1.C, SW1G$2.1, SW2G$1.C, SW2G$2.1; no longer CONN_LCD.2, U$14.S1, U$14.S2
- net LCD_B-: now also LCD1.K; no longer CONN_LCD.15
- net LCD_D0: now also LCD1.DB0; no longer CONN_LCD.8
- net LCD_D1: now also LCD1.DB1; no longer CONN_LCD.7
- net LCD_D2: now also LCD1.DB2; no longer CONN_LCD.10
- net LCD_D3: now also LCD1.DB3; no longer CONN_LCD.9
- net LCD_D4: now also LCD1.DB4; no longer CONN_LCD.12
- net LCD_D5: now also LCD1.DB5; no longer CONN_LCD.11
- net LCD_D6: now also LCD1.DB6; no longer CONN_LCD.14
- net LCD_D7: now also LCD1.DB7; no longer CONN_LCD.13
- net LCD_E1: now also LCD1.E; no longer CONN_LCD.5
- net LCD_RS: now also LCD1.RS; no longer CONN_LCD.3
- net LCD_RW: now also LCD1.R/W; no longer CONN_LCD.6
- net LCD_V0: now also LCD1.V5; no longer CONN_LCD.4
- net LCD_VD: now also LCD1.VDD; no longer CONN_LCD.1
- net SCL: now also C26.P$2
- net SDA: now also C27.P$2
Other:
- note added: "USB_VBUS"

Commit message: wip
Parts:
- removed C3: 1uF, microbuilder:CAP_CERAMIC0603
Connections:
- net 3.3V: no longer C3.P$2
- net GND: no longer C3.P$1
- net N$10: now also PRTR5V0U2X1.D1
- net USB_DM: no longer PRTR5V0U2X1.D1
Other:
- moved on the sheet: R6
Changed lines of the file:
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@@
 <setting verticaltext="up"/>
 </settings>
-<grid distance="0.1" unitdist="inch" unit="inch" style="lines" multiple="1" display="no" altdistance="0.01" altunitdist="inch" altunit="inch"/>
+<grid distance="0.05" unitdist="inch" unit="inch" style="lines" multiple="1" display="no" altdistance="0.01" altunitdist="inch" altunit="inch"/>
 <layers>
 <layer number="1" name="Top" color="4" fill="1" visible="no" active="no"/>
@@
 <part name="U$4" library="microbuilder" deviceset="GND" device=""/>
 <part name="U$5" library="microbuilder" deviceset="3.3V" device=""/>
-<part name="C3" library="microbuilder" deviceset="CAP_CERAMIC" device="0603" value="1uF"/>
-<part name="U$6" library="microbuilder" deviceset="GND" device=""/>
 <part name="C4" library="microbuilder" deviceset="CAP_CERAMIC" device="0603" value="0.1uF"/>
 <part name="C5" library="microbuilder" deviceset="CAP_CERAMIC" device="0603" value="0.1uF"/>
@@
 <instance part="U$4" gate="G$1" x="12.7" y="137.16"/>
 <instance part="U$5" gate="G$1" x="5.08" y="111.76" rot="R90"/>
-<instance part="C3" gate="G$1" x="12.7" y="109.22" rot="R180"/>
-<instance part="U$6" gate="G$1" x="12.7" y="99.06"/>
 <instance part="C4" gate="G$1" x="22.86" y="162.56"/>
 <instance part="C5" gate="G$1" x="12.7" y="162.56"/>
@@
 <instance part="U$16" gate="G$1" x="-41.91" y="185.42"/>
 <instance part="U$17" gate="G$1" x="-44.45" y="193.04" rot="R90"/>
-<instance part="R6" gate="G$1" x="5.08" y="195.58" rot="R180"/>
+<instance part="R6" gate="G$1" x="-5.08" y="195.58" rot="R180"/>
 <instance part="R7" gate="G$1" x="-6.35" y="198.12" rot="R180"/>
 <instance part="C18" gate="G$1" x="44.45" y="190.5"/>
@@
 <pinref part="STM32F407XX1" gate="G$1" pin="VBAT"/>
 <pinref part="U$5" gate="G$1" pin="3.3V"/>
-<wire x1="7.62" y1="111.76" x2="12.7" y2="111.76" width="0.1524" layer="91"/>
-<pinref part="C3" gate="G$1" pin="P$2"/>
-<wire x1="12.7" y1="111.76" x2="35.56" y2="111.76" width="0.1524" layer="91"/>
-<junction x="12.7" y="111.76"/>
+<wire x1="7.62" y1="111.76" x2="35.56" y2="111.76" width="0.1524" layer="91"/>
 </segment>
 <segment>
@@
 <wire x1="12.7" y1="139.7" x2="15.24" y2="139.7" width="0.1524" layer="91"/>
 <junction x="12.7" y="139.7"/>
-</segment>
-<segment>
-<pinref part="C3" gate="G$1" pin="P$1"/>
-<pinref part="U$6" gate="G$1" pin="GND"/>
-<wire x1="12.7" y1="101.6" x2="12.7" y2="104.14" width="0.1524" layer="91"/>
 </segment>
 <segment>
@@
 <pinref part="U$14" gate="G$1" pin="D-"/>
 <pinref part="R6" gate="G$1" pin="1"/>
-<wire x1="19.05" y1="195.58" x2="10.16" y2="195.58" width="0.1524" layer="91"/>
+<wire x1="19.05" y1="195.58" x2="5.08" y2="195.58" width="0.1524" layer="91"/>
+<pinref part="PRTR5V0U2X1" gate="G$1" pin="D1"/>
+<wire x1="5.08" y1="195.58" x2="0" y2="195.58" width="0.1524" layer="91"/>
+<wire x1="-19.05" y1="208.28" x2="-19.05" y2="203.2" width="0.1524" layer="91"/>
+<wire x1="-19.05" y1="203.2" x2="5.08" y2="203.2" width="0.1524" layer="91"/>
+<wire x1="5.08" y1="203.2" x2="5.08" y2="195.58" width="0.1524" layer="91"/>
+<junction x="5.08" y="195.58"/>
 </segment>
 </net>
@@
 <segment>
 <pinref part="R6" gate="G$1" pin="2"/>
-<wire x1="0" y1="195.58" x2="-19.05" y2="195.58" width="0.1524" layer="91"/>
-<wire x1="-19.05" y1="195.58" x2="-40.64" y2="195.58" width="0.1524" layer="91"/>
+<wire x1="-10.16" y1="195.58" x2="-40.64" y2="195.58" width="0.1524" layer="91"/>
 <label x="-40.64" y="195.58" size="1.778" layer="95"/>
-<pinref part="PRTR5V0U2X1" gate="G$1" pin="D1"/>
-<wire x1="-19.05" y1="208.28" x2="-19.05" y2="195.58" width="0.1524" layer="91"/>
-<junction x="-19.05" y="195.58"/>
-</segment>
-<segment>
+</segment>
+<segment>

Commit message: wip
Connections:
- net N$3 renamed VREF
- net N$4 renamed VDDA
Changed lines of the file:
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@@
 </segment>
 </net>
-<net name="N$3" class="0">
+<net name="VREF" class="0">
 <segment>
 <pinref part="STM32F407XX1" gate="G$1" pin="VREF+"/>
@@
 </segment>
 </net>
-<net name="N$4" class="0">
+<net name="VDDA" class="0">
 <segment>
 <wire x1="10.16" y1="127" x2="10.16" y2="134.62" width="0.1524" layer="91"/>

Commit message: wip
Parts:
- removed C19: 100uF, microbuilder:CAP_ELECTROLYTICPANASONIC_D
- renumbered LED3 to LED_PWR
Connections:
- net USB_DM renamed USB_D_N
- net USB_DP renamed USB_D_PP
- net 3.3V: no longer C19.+
- net GND: no longer C19.-
Changed lines of the file:
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@@
 <part name="JTAG" library="microbuilder" deviceset="HEADER-1X6" device="ROUND"/>
 <part name="U$24" library="microbuilder" deviceset="3.3V" device=""/>
-<part name="C19" library="microbuilder" deviceset="CAP_ELECTROLYTIC" device="PANASONIC_D" value="100uF"/>
 <part name="U$25" library="keves" deviceset="MIC37100" device=""/>
 <part name="U$26" library="microbuilder" deviceset="5.0V" device=""/>
@@
 <part name="C22" library="microbuilder" deviceset="CAP_CERAMIC" device="0603" value="0.1uF"/>
 <part name="R3" library="microbuilder" deviceset="RESISTOR" device="0603" value="680"/>
-<part name="LED3" library="microbuilder" deviceset="LED" device="0603"/>
+<part name="LED_PWR" library="microbuilder" deviceset="LED" device="0603"/>
 <part name="U$29" library="microbuilder" deviceset="GND" device=""/>
 <part name="U1" library="microbuilder" deviceset="EEPROM_I2C_SOIC8_GENERIC" device="" value="24LC512"/>
@@
 <instance part="JTAG" gate="A" x="162.56" y="191.77" rot="MR0"/>
 <instance part="U$24" gate="G$1" x="194.31" y="199.39" rot="R270"/>
-<instance part="C19" gate="G$1" x="-62.23" y="162.56"/>
 <instance part="U$25" gate="G$1" x="-99.06" y="200.66"/>
 <instance part="U$26" gate="G$1" x="-125.73" y="200.66" rot="R90"/>
@@
 <instance part="C22" gate="G$1" x="-66.04" y="193.04"/>
 <instance part="R3" gate="G$1" x="-54.61" y="195.58" rot="R90"/>
-<instance part="LED3" gate="G$1" x="-54.61" y="182.88" rot="R270"/>
+<instance part="LED_PWR" gate="G$1" x="-54.61" y="182.88" rot="R270"/>
 <instance part="U$29" gate="G$1" x="-54.61" y="175.26"/>
 <instance part="U1" gate="G$1" x="-110.49" y="132.08"/>
@@
 <junction x="-38.1" y="167.64"/>
 <wire x1="-38.1" y1="167.64" x2="-48.26" y2="167.64" width="0.1524" layer="91"/>
-<pinref part="C19" gate="G$1" pin="+"/>
-<wire x1="-48.26" y1="167.64" x2="-62.23" y2="167.64" width="0.1524" layer="91"/>
-<junction x="-48.26" y="167.64"/>
 </segment>
 <segment>
@@
 <pinref part="C5" gate="G$1" pin="P$2"/>
 <junction x="12.7" y="160.02"/>
-<pinref part="C19" gate="G$1" pin="-"/>
-<wire x1="-62.23" y1="160.02" x2="-48.26" y2="160.02" width="0.1524" layer="91"/>
 </segment>
 <segment>
@@
 </segment>
 <segment>
-<pinref part="LED3" gate="G$1" pin="C"/>
+<pinref part="LED_PWR" gate="G$1" pin="C"/>
 <pinref part="U$29" gate="G$1" pin="GND"/>
 <wire x1="-54.61" y1="177.8" x2="-54.61" y2="180.34" width="0.1524" layer="91"/>
@@
 </segment>
 </net>
-<net name="USB_DM" class="0">
-<segment>
-<pinref part="R6" gate="G$1" pin="2"/>
-<wire x1="-10.16" y1="195.58" x2="-40.64" y2="195.58" width="0.1524" layer="91"/>
-<label x="-40.64" y="195.58" size="1.778" layer="95"/>
-</segment>
-<segment>
-<pinref part="STM32F407XX1" gate="G$1" pin="PA11"/>
-<wire x1="177.8" y1="137.16" x2="184.15" y2="137.16" width="0.1524" layer="91"/>
-<label x="182.88" y="137.16" size="1.778" layer="95"/>
-</segment>
-</net>
-<net name="USB_DP" class="0">
+<net name="USB_D_PP" class="0">
 <segment>
 <pinref part="R7" gate="G$1" pin="2"/>
@@
 <segment>
 <pinref part="R3" gate="G$1" pin="1"/>
-<pinref part="LED3" gate="G$1" pin="A"/>
+<pinref part="LED_PWR" gate="G$1" pin="A"/>
 <wire x1="-54.61" y1="190.5" x2="-54.61" y2="187.96" width="0.1524" layer="91"/>
 </segment>
@@
 </segment>
 </net>
+<net name="USB_D_N" class="0">
+<segment>
+<pinref part="R6" gate="G$1" pin="2"/>
+<wire x1="-10.16" y1="195.58" x2="-40.64" y2="195.58" width="0.1524" layer="91"/>
+<label x="-40.64" y="195.58" size="1.778" layer="95"/>
+</segment>
+<segment>
+<pinref part="STM32F407XX1" gate="G$1" pin="PA11"/>
+<wire x1="177.8" y1="137.16" x2="184.15" y2="137.16" width="0.1524" layer="91"/>
+<label x="182.88" y="137.16" size="1.778" layer="95"/>
+</segment>
+</net>

Commit message: wip
Parts:
- C24: value 100nF -> 0.1uF
Connections:
- net SCS_D10: now also R36.1, S3.P, S3.P1; no longer SW2G$2.2
- net SCS_D5: now also SW2G$2.2; no longer R36.1, S3.P, S3.P1
- net SCS_D6: now also SW2G$1.A; no longer R37.1, S4.P, S4.P1
- net SCS_D7: now also SW2G$1.B; no longer R38.1, S5.P, S5.P1
- net SCS_D8: now also R38.1, S5.P, S5.P1; no longer SW2G$1.B
- net SCS_D9: now also R37.1, S4.P, S4.P1; no longer SW2G$1.A
Changed lines of the file:
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@@
 <part name="U$64" library="microbuilder" deviceset="3.3V" device=""/>
 <part name="IC5" library="74xx-eu" deviceset="74*595" device="D" technology="HC"/>
-<part name="C24" library="microbuilder" deviceset="CAP_CERAMIC" device="0603" value="100nF"/>
+<part name="C24" library="microbuilder" deviceset="CAP_CERAMIC" device="0603" value="0.1uF"/>
 <part name="U$67" library="microbuilder" deviceset="GND" device=""/>
 <part name="R20" library="microbuilder" deviceset="RESISTOR" device="_0603" value="1K"/>
@@
 </segment>
 </net>
-<net name="SCS_D5" class="0">
+<net name="SCS_D8" class="0">
+<segment>
+<wire x1="157.48" y1="106.68" x2="160.02" y2="106.68" width="0.1524" layer="91"/>
+<junction x="157.48" y="106.68"/>
+<pinref part="S5" gate="1" pin="P"/>
+<pinref part="S5" gate="1" pin="P1"/>
+<pinref part="R38" gate="G$1" pin="1"/>
+<wire x1="157.48" y1="106.68" x2="144.78" y2="106.68" width="0.1524" layer="91"/>
+<label x="142.24" y="106.68" size="1.778" layer="95"/>
+</segment>
+</net>
+<net name="SCS_D9" class="0">
+<segment>
+<wire x1="134.62" y1="106.68" x2="137.16" y2="106.68" width="0.1524" layer="91"/>
+<junction x="134.62" y="106.68"/>
+<pinref part="S4" gate="1" pin="P"/>
+<pinref part="S4" gate="1" pin="P1"/>
+<pinref part="R37" gate="G$1" pin="1"/>
+<wire x1="134.62" y1="106.68" x2="121.92" y2="106.68" width="0.1524" layer="91"/>
+<label x="119.38" y="106.68" size="1.778" layer="95"/>
+</segment>
+</net>
+<net name="SCS_D10" class="0">
 <segment>
 <wire x1="109.22" y1="106.68" x2="111.76" y2="106.68" width="0.1524" layer="91"/>
@@
 </segment>
 </net>
-<net name="SCS_D6" class="0">
-<segment>
-<wire x1="134.62" y1="106.68" x2="137.16" y2="106.68" width="0.1524" layer="91"/>
-<junction x="134.62" y="106.68"/>
-<pinref part="S4" gate="1" pin="P"/>
-<pinref part="S4" gate="1" pin="P1"/>
-<pinref part="R37" gate="G$1" pin="1"/>
-<wire x1="134.62" y1="106.68" x2="121.92" y2="106.68" width="0.1524" layer="91"/>
-<label x="119.38" y="106.68" size="1.778" layer="95"/>
+<net name="A0" class="0">
+<segment>
+<pinref part="R39" gate="G$1" pin="S"/>
+<wire x1="187.96" y1="101.6" x2="187.96" y2="93.98" width="0.1524" layer="91"/>
+<label x="187.96" y="93.98" size="1.778" layer="95" rot="R90"/>
+</segment>
+</net>
+<net name="A1" class="0">
+<segment>
+<pinref part="R40" gate="G$1" pin="S"/>
+<wire x1="220.98" y1="101.6" x2="220.98" y2="93.98" width="0.1524" layer="91"/>
+<label x="220.98" y="93.98" size="1.778" layer="95" rot="R90"/>
+</segment>
+</net>
+<net name="A2" class="0">
+<segment>
+<pinref part="R41" gate="G$1" pin="S"/>
+<wire x1="254" y1="101.6" x2="254" y2="93.98" width="0.1524" layer="91"/>
+<label x="254" y="93.98" size="1.778" layer="95" rot="R90"/>
+</segment>
+</net>
+<net name="A3" class="0">
+<segment>
+<pinref part="R42" gate="G$1" pin="S"/>
+<wire x1="287.02" y1="101.6" x2="287.02" y2="93.98" width="0.1524" layer="91"/>
+<label x="287.02" y="93.98" size="1.778" layer="95" rot="R90"/>
+</segment>
+</net>
+<net name="A4" class="0">
+<segment>
+<pinref part="R43" gate="G$1" pin="S"/>
+<wire x1="320.04" y1="101.6" x2="320.04" y2="93.98" width="0.1524" layer="91"/>
+<label x="320.04" y="93.98" size="1.778" layer="95" rot="R90"/>
 </segment>
 </net>
 <net name="SCS_D7" class="0">
-<segment>
-<wire x1="157.48" y1="106.68" x2="160.02" y2="106.68" width="0.1524" layer="91"/>
-<junction x="157.48" y="106.68"/>
-<pinref part="S5" gate="1" pin="P"/>
-<pinref part="S5" gate="1" pin="P1"/>
-<pinref part="R38" gate="G$1" pin="1"/>
-<wire x1="157.48" y1="106.68" x2="144.78" y2="106.68" width="0.1524" layer="91"/>
-<label x="142.24" y="106.68" size="1.778" layer="95"/>
-</segment>
-</net>
-<net name="SCS_D8" class="0">
 <segment>
 <wire x1="73.66" y1="25.4" x2="88.9" y2="25.4" width="0.1524" layer="91"/>
@@
 </segment>
 </net>
-<net name="SCS_D9" class="0">
+<net name="SCS_D6" class="0">
 <segment>
 <wire x1="73.66" y1="22.86" x2="86.36" y2="22.86" width="0.1524" layer="91"/>
@@
 </segment>
 </net>
-<net name="SCS_D10" class="0">
+<net name="SCS_D5" class="0">
 <segment>
 <wire x1="73.66" y1="27.94" x2="83.82" y2="27.94" width="0.1524" layer="91"/>
@@
 </segment>
 </net>
-<net name="A0" class="0">
-<segment>
-<pinref part="R39" gate="G$1" pin="S"/>
-<wire x1="187.96" y1="101.6" x2="187.96" y2="93.98" width="0.1524" layer="91"/>
-<label x="187.96" y="93.98" size="1.778" layer="95" rot="R90"/>
-</segment>
-</net>
-<net name="A1" class="0">
-<segment>
-<pinref part="R40" gate="G$1" pin="S"/>
-<wire x1="220.98" y1="101.6" x2="220.98" y2="93.98" width="0.1524" layer="91"/>
-<label x="220.98" y="93.98" size="1.778" layer="95" rot="R90"/>
-</segment>
-</net>
-<net name="A2" class="0">
-<segment>
-<pinref part="R41" gate="G$1" pin="S"/>
-<wire x1="254" y1="101.6" x2="254" y2="93.98" width="0.1524" layer="91"/>
-<label x="254" y="93.98" size="1.778" layer="95" rot="R90"/>
-</segment>
-</net>
-<net name="A3" class="0">
-<segment>
-<pinref part="R42" gate="G$1" pin="S"/>
-<wire x1="287.02" y1="101.6" x2="287.02" y2="93.98" width="0.1524" layer="91"/>
-<label x="287.02" y="93.98" size="1.778" layer="95" rot="R90"/>
-</segment>
-</net>
-<net name="A4" class="0">
-<segment>
-<pinref part="R43" gate="G$1" pin="S"/>
-<wire x1="320.04" y1="101.6" x2="320.04" y2="93.98" width="0.1524" layer="91"/>
-<label x="320.04" y="93.98" size="1.778" layer="95" rot="R90"/>
-</segment>
-</net>

Commit message: wip
Parts:
- removed C11: 0.1uF, microbuilder:CAP_CERAMIC0603
Connections:
- net 3.3V: no longer C11.P$1
- net GND: no longer C11.P$2
- net SCS_D0: now also SW2G$1.B; no longer SW1G$1.B
- net SCS_D1: now also SW2G$1.A; no longer SW1G$1.A
- net SCS_D3: now also SW1G$1.B; no longer R34.1, S1.P, S1.P1
- net SCS_D4: now also SW1G$1.A; no longer R35.1, S2.P, S2.P1
- net SCS_D6: now also R35.1, S2.P, S2.P1; no longer SW2G$1.A
- net SCS_D7: now also R34.1, S1.P, S1.P1; no longer SW2G$1.B
