File: eagle/rev_b/cpu_eval_board.sch (EAGLE design)
At the start: 105 parts, among them IC1 6N138S-TA1, IC2 6N138S-TA1, IC5 74HC595D, Q1 BC337, SW1 Encoder, SW2 Encoder, U1 24LC512, Y1 8MHz

Commit message: all routed
Parts:
- added C3: 0.1uF, microbuilder:CAP_CERAMIC0603
- added FLASH1: AT25DF641A or MX25L6406E, vovtech:FLASH-SPI
- added SPI_A: (no value), pinhead:PINHD-2X6
- added SPI_B: (no value), pinhead:PINHD-2X7
Connections:
- removed net SWO: R16.2, STM32F407XX1.PB3
- new net A_RC1: SPI_A.12, STM32F407XX1.PB12
- new net A_RC2: SPI_A.11, STM32F407XX1.PD10
- new net A_SC: SPI_A.10, SPI_A.9, STM32F407XX1.PB13
- new net A_SI: SPI_A.7, STM32F407XX1.PB14
- new net A_SO: SPI_A.8, STM32F407XX1.PB15
- new net B_RC1: SPI_B.12, STM32F407XX1.PA15
- new net B_RC2: SPI_B.11, STM32F407XX1.PB8
- new net B_RC3: SPI_B.14, STM32F407XX1.PC0
- new net B_RC4: SPI_B.13, STM32F407XX1.PC3
- new net B_RC5: FLASH1.#CS, STM32F407XX1.PE5
- new net B_SC: FLASH1.SCLK, R16.2, SPI_B.10, SPI_B.9, STM32F407XX1.PB3
- new net B_SI: FLASH1.SO/IO1, SPI_B.7, STM32F407XX1.PB4
- new net B_SO: FLASH1.SI/IO0, SPI_B.8, STM32F407XX1.PB5
- net 3.3V: now also C3.P$2, FLASH1.#HOLD/IO3, FLASH1.#WP/ACC/IO2, FLASH1.VCC, SPI_A.5, SPI_A.6, SPI_B.5, SPI_B.6
- net 5.0V: now also SPI_A.1, SPI_A.2, SPI_B.1, SPI_B.2
- net GND: now also C3.P$1, FLASH1.GND, SPI_A.3, SPI_A.4, SPI_B.3, SPI_B.4

Commit message: before silkscreen edits
Parts:
- added R44, R45: 10K, microbuilder:RESISTOR0603
- added R46: 0, microbuilder:RESISTOR0603
Connections:
- new net N$3: R46.1, STM32F407XX1.PA9
- net 3.3V: now also R44.2
- net 5.0V: now also R46.2; no longer STM32F407XX1.PA9
- net BOOT1: now also R45.1
- net GND: now also R45.2
- net NRST: now also R44.1
Changed lines of the file:
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@@
 <part name="U$93" library="microbuilder" deviceset="3.3V" device=""/>
 <part name="U$94" library="microbuilder" deviceset="3.3V" device=""/>
+<part name="R44" library="microbuilder" deviceset="RESISTOR" device="0603" value="10K"/>
+<part name="U$95" library="microbuilder" deviceset="3.3V" device=""/>
+<part name="R45" library="microbuilder" deviceset="RESISTOR" device="0603" value="10K"/>
+<part name="U$96" library="microbuilder" deviceset="GND" device=""/>
+<part name="R46" library="microbuilder" deviceset="RESISTOR" device="0603" value="0"/>
 </parts>
 <sheets>
 <sheet>
 <plain>
-<text x="182.88" y="133.35" size="1.778" layer="97">USB_VBUS</text>
+<text x="199.39" y="133.35" size="1.778" layer="97">USB_VBUS</text>
 </plain>
 <instances>
@@
 <instance part="U$33" gate="G$1" x="-130.81" y="119.38"/>
 <instance part="U$34" gate="G$1" x="-138.43" y="119.38"/>
-<instance part="U$35" gate="G$1" x="185.42" y="132.08" rot="R270"/>
+<instance part="U$35" gate="G$1" x="203.2" y="132.08" rot="R270"/>
 <instance part="H1" gate="G$1" x="-167.64" y="193.04"/>
 <instance part="H2" gate="G$1" x="-167.64" y="187.96"/>
@@
 <instance part="U$93" gate="G$1" x="-83.82" y="11.43" rot="R90"/>
 <instance part="U$94" gate="G$1" x="-59.69" y="11.43" rot="R270"/>
+<instance part="R44" gate="G$1" x="44.45" y="204.47" rot="R90"/>
+<instance part="U$95" gate="G$1" x="44.45" y="214.63"/>
+<instance part="R45" gate="G$1" x="15.24" y="60.96" rot="R90"/>
+<instance part="U$96" gate="G$1" x="15.24" y="71.12" rot="R180"/>
+<instance part="R46" gate="G$1" x="191.77" y="132.08"/>
 </instances>
 <busses>
@@
 <wire x1="-81.28" y1="11.43" x2="-74.93" y2="11.43" width="0.1524" layer="91"/>
 </segment>
+<segment>
+<pinref part="R44" gate="G$1" pin="2"/>
+<pinref part="U$95" gate="G$1" pin="3.3V"/>
+<wire x1="44.45" y1="209.55" x2="44.45" y2="212.09" width="0.1524" layer="91"/>
+</segment>
 </net>
 <net name="GND" class="0">
@@
 <wire x1="-62.23" y1="13.97" x2="-67.31" y2="13.97" width="0.1524" layer="91"/>
 </segment>
+<segment>
+<pinref part="R45" gate="G$1" pin="2"/>
+<pinref part="U$96" gate="G$1" pin="GND"/>
+<wire x1="15.24" y1="68.58" x2="15.24" y2="66.04" width="0.1524" layer="91"/>
+</segment>
 </net>
 <net name="N$1" class="0">
@@
 <segment>
 <pinref part="STM32F407XX1" gate="G$1" pin="PB2"/>
-<wire x1="35.56" y1="55.88" x2="7.62" y2="55.88" width="0.1524" layer="91"/>
+<wire x1="35.56" y1="55.88" x2="15.24" y2="55.88" width="0.1524" layer="91"/>
 <pinref part="R5" gate="G$1" pin="1"/>
+<wire x1="15.24" y1="55.88" x2="7.62" y2="55.88" width="0.1524" layer="91"/>
 <wire x1="7.62" y1="55.88" x2="1.27" y2="55.88" width="0.1524" layer="91"/>
 <junction x="7.62" y="55.88"/>
 <label x="-3.81" y="55.88" size="1.778" layer="95"/>
+<pinref part="R45" gate="G$1" pin="1"/>
+<junction x="15.24" y="55.88"/>
 </segment>
 </net>
@@
 </segment>
 <segment>
-<pinref part="STM32F407XX1" gate="G$1" pin="PA9"/>
-<wire x1="177.8" y1="132.08" x2="182.88" y2="132.08" width="0.1524" layer="91"/>
 <pinref part="U$35" gate="G$1" pin="5.0V"/>
+<pinref part="R46" gate="G$1" pin="2"/>
+<wire x1="196.85" y1="132.08" x2="200.66" y2="132.08" width="0.1524" layer="91"/>
 </segment>
 <segment>
@@
 <junction x="55.88" y="196.85"/>
 <label x="36.83" y="196.85" size="1.778" layer="95"/>
+<wire x1="44.45" y1="196.85" x2="44.45" y2="199.39" width="0.1524" layer="91"/>
+<pinref part="R44" gate="G$1" pin="1"/>
 </segment>
 <segment>
@@
 </segment>
 </net>
+<net name="N$3" class="0">
+<segment>
+<pinref part="R46" gate="G$1" pin="1"/>
+<pinref part="STM32F407XX1" gate="G$1" pin="PA9"/>
+<wire x1="186.69" y1="132.08" x2="177.8" y2="132.08" width="0.1524" layer="91"/>
+</segment>
+</net>

Commit message: bom
Parts:
- C1, C2: PARTNO (none) -> GRM188R61E225KA12D,Murata Electronics,,81-GRM188R61E225KA2D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
- C10, C12, C13, C18, C22, C23, C24, C3, C4, C5, C6, C7, C8, C9: PARTNO (none) -> VJ0603Y104JXJPW1BC,Vishay / Vitramon,,77-VJ0603Y104JXJPBC,M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
- C14, C15: PARTNO (none) -> GRM188R61E105KA12D,Murata Electronics,,81-GRM188R61E105KA12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
- C16, C17: PARTNO (none) -> GRM1885C1H200JA01D,Murata Electronics,,81-GRM39C200J50,Mult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
- C20, C21: PARTNO (none) -> GRM21BR71A106KA73L,Murata Electronics,,81-GRM21BR71A106KA3L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
- C25: PARTNO (none) -> CGA3E3X7S2A104M080AB,TDK,,810-CGA3E3X7S2A104AB,Multilayer C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
- C26, C27: PARTNO (none) -> VJ0603A180JXACW1BC,Vishay / Vitramon,,77-VJ0603A180JXACBC,M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
- D1, D2: PARTNO (none) -> 1N4148WSFL-G3-08,Vishay Semiconductors,,78-1N4148WSFL-G3-08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
- FB1: PARTNO (none) -> HZ0805E601R-10,Laird Technologies,,875-HZ0805E601R-10,"EMI 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
- IC1, IC2: PARTNO (none) -> 6N138S-TA1,Lite-On,,859-6N138STA1,High Speed Optocouplers D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
- IC5: PARTNO (none) -> 74HC595D,NXP Semiconductors,,771-74HC595D-T,Counter Shift R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
- JP2: PARTNO (none) -> 4-103327-5,TE Connectivity / AMP,,571-4-103327-5,3 pin head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
- JTAG: PARTNO (none) -> XG8V-0641,Omron Electronics,,653-XG8V-0641,6 pin header 1 r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
- LCD1: PARTNO (none) -> NHD-C0220AA-FSW-FTW,Newhaven Display,,763-C0220AA-FSW-FTW,L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
- LCD_POT1, LCD_POT2: PARTNO (none) -> 67WR10KLF,BI Technologies / TT Electronics,,858-67WR10KLF,"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
- LED1, LED2, LED_PWR: PARTNO (none) -> VLMS1300-GS08,Vishay Semiconductors,,78-VLMS1300-GS08,Stand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
- MIDI_IN1, MIDI_IN2, MIDI_OUT1, MIDI_OUT2: PARTNO (none) -> 57PC5F,Switchcraft,,502-57PC5F,DIN Connectors 5 COND 180 DI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
- PRTR5V0U2X1: PARTNO (none) -> PRTR5V0U2X,215",NXP Semiconductors,,771-PRTR5V0U2X-T/R,ESD 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
- Q1: PARTNO (none) -> BC337-16 A1,Taiwan ,,821-BC337-16-A1,Bipolar Transistors - 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
- R1: PARTNO (none) -> CRCW060347R0FKEA,Vishay / Dale,,71-CRCW0603-47-E3,Thick Fil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
- R10, R11, R3: PARTNO (none) -> MCT06030C6800FP500,Vishay / Beyschlag,,594-MCT06030C6800FP5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
- R12, R14, R15, R16, R4, R46: PARTNO (none) -> MCT06030Z0000ZP500,Vishay / Beyschlag,,594-MCT06030Z0000ZP5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
- R13, R17: PARTNO (none) -> MCT06030C2201FP500,Vishay / Beyschlag,,594-MCT06030C2201FP5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
- R18, R34, R35, R36, R37, R38, R44, R45, R5: PARTNO (none) -> CRCW060310K0FKEA,Vishay / Dale,,71-CRCW0603-10K-E3,Thick Fi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
- R19, R20, R21, R22, R28, R33: PARTNO (none) -> CRCW06031K00FKEA,Vishay / Dale,,71-CRCW0603-1.0K-E3,Thick F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
- R2: PARTNO (none) -> RT0603FRE07510RL,Yageo,,603-RT0603FRE07510RL,Thin Film Resi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
- R23: PARTNO (none) -> CRCW06031M00FKEA,Vishay / Dale,,71-CRCW0603-1.0M-E3,Thick F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
- R24, R25, R26, R29, R30, R31: PARTNO (none) -> MCT06030C2200FP500,Vishay / Beyschlag,,594-MCT06030C2200FP5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
- R27, R32: PARTNO (none) -> MCT06030C4701FP500,Vishay,,594-MCT06030C4701FP5,Thin Film R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
- R39, R40, R41, R42, R43, SW1, SW2: PARTNO (none) -> RK09D1130C2P,ALPS,,688-RK09D1130C2P,Potentiometers 9MM 10K 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
- R6, R7: PARTNO (none) -> MCT06030C2209FP500,Vishay / Beyschlag,,594-MCT06030C2209FP5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
- R8: PARTNO (none) -> RT0603FRE07330RL,Yageo,,603-RT0603FRE07330RL,Thin Film Resi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
- R9: PARTNO (none) -> RT0603FRE07220KL,Yageo,,603-RT0603FRE07220KL,Thin Film Resi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
- S1, S2, S3, S4, S5: PARTNO (none) -> TL1100F160Q,E-Switch,,612-TL1100,Tactile Switches 12X7.3MM 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
- SPI_A: PARTNO (none) -> 67996-412HLF,FCI,,649-67996-412HLF,6x2 header pins, REF4
- SPI_B: PARTNO (none) -> 67997-414HLF,FCI,,649-67997-414HLF,7x2 header pins, REF5
- STM32F407XX1: PARTNO (none) -> STM32F407VGT6,ST,,511-STM32F407VGT6,ARM Microcontrollers - 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
- SW_RST, SW_USER: PARTNO (none) -> EVQ-PQHB55,Panasonic,,667-EVQ-PQHB55,Tactile Switches Super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
- U$14: PARTNO (none) -> 67068-9001,Molex,,538-67068-9001,USB Connectors USB Type B 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
- U$25: PARTNO (none) -> MIC37100-3.3WS TR,Micrel,,998-MIC37100-3.3WSTR,LDO Voltage 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
- U1: PARTNO (none) -> 24LC512-I/SN,Microchip Technology,,579-24LC512-I/SN,EEPROM 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
- Y1: PARTNO (none) -> ABLS-8.000MHZ-B4-T,ABRACON,,815-ABLS-8.0M-T,Crystals 8.000M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
