File: eagle/rev_b/cpu_eval_board.brd (EAGLE design)
At the start: 114.3 x 101.6 mm, 108 parts, among them IC1 6N138S-TA1, IC2 6N138S-TA1, IC5 74HC595D, Q1 BC337, SW1 Encoder, SW2 Encoder, U1 24LC512, Y1 8MHz

Commit message: wip
Parts:
- removed C3: 1uF, microbuilder:0603
- moved STM32F407XX1 253.1 mm to (102.6, 61.7)
- moved IC2 167.1 mm to (54.6, 74.9), turned to 270 degrees
- moved R39 165.1 mm to (10.2, -121.9)
- moved R40 165.1 mm to (33.7, -121.9)
- moved R42 165.1 mm to (80.6, -121.9)
- moved R43 165.1 mm to (104.1, -121.9)
- moved C10 164.5 mm to (103.1, 69.1), flipped to the bottom
- moved C17 163.7 mm to (107.4, 50.5), turned to 90 degrees
- moved C7 160.2 mm to (104.1, 59.2), flipped to the bottom, turned to 90 degrees
- moved C2 159.2 mm to (104.4, 65.8), flipped to the bottom, turned to 90 degrees
- moved R6 158.3 mm to (97.0, 79.0), turned to 270 degrees
- moved C8 156.8 mm to (94.4, 58.2), flipped to the bottom, turned to 90 degrees
- moved Y1 156.2 mm to (99.8, 47.5)
- moved IC1 154.0 mm to (14.0, 76.2), turned to 270 degrees
- moved C6 152.2 mm to (102.5, 59.2), flipped to the bottom, turned to 90 degrees
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Connections:
- net 3.3V: no longer C3.2
- net GND: no longer C3.1
- net N$10: now also PRTR5V0U2X1.P$2
- net USB_DM: no longer PRTR5V0U2X1.P$2
Routing:
- net 3.3V: track 0.00 -> 24.0 mm, vias 0 -> 7
- net GND: track 0.00 -> 9.95 mm, vias 0 -> 5
- net N$1: track 0.00 -> 3.84 mm, vias 0 -> 1
- net N$2: track 0.00 -> 3.15 mm, vias 0 -> 1
- added copper zone on layer 1, net 3.3V
- added copper zone on layer 16, net GND

Commit message: wip
Parts:
- moved C15 143.8 mm to (100.6, 59.7), flipped to the bottom, turned to 90 degrees
- moved C14 142.5 mm to (105.7, 60.5), flipped to the bottom, turned to 270 degrees
- moved FB1 135.0 mm to (100.6, 62.7), flipped to the bottom, turned to 180 degrees
- moved C13 132.7 mm to (102.2, 59.7), flipped to the bottom, turned to 270 degrees
- moved R1 128.5 mm to (98.9, 59.7), flipped to the bottom, turned to 270 degrees
- moved C12 128.1 mm to (104.0, 60.5), flipped to the bottom, turned to 90 degrees
- moved C7 3.54 mm to (107.4, 60.5)
- moved C6 3.41 mm to (101.0, 56.1), turned to 270 degrees
- moved C5 0.74 mm to (97.3, 59.7)
- moved C4 0.63 mm to (95.6, 59.7)
- moved C8 0.40 mm to (94.0, 58.3)
Connections:
- net N$3 renamed VREF
- net N$4 renamed VDDA
Routing:
- net VDDA: track 0.00 -> 18.7 mm, vias 0 -> 3
- net VREF: track 0.00 -> 7.19 mm, vias 0 -> 1
- net 3.3V: track 24.0 -> 28.4 mm, vias 7 -> 8
- net GND: track 9.95 -> 12.1 mm

Commit message: wip
Parts:
- removed C19: 100uF, microbuilder:PANASONIC_D
- removed LED3: (no value), microbuilder:CHIPLED_0603
- added LED_PWR: (no value), microbuilder:CHIPLED_0603
- moved C26 204.6 mm to (137.3, 38.9), turned to 90 degrees
- moved C27 203.0 mm to (135.1, 38.7), turned to 90 degrees
- moved R31 201.9 mm to (86.7, 85.7), turned to 90 degrees
- moved R29 195.0 mm to (67.4, 86.2), turned to 180 degrees
- moved R30 194.2 mm to (71.1, 85.2), turned to 90 degrees
- moved R13 190.4 mm to (133.7, 46.0), turned to 90 degrees
- moved R26 189.5 mm to (46.7, 86.1), turned to 180 degrees
- moved R23 182.7 mm to (91.7, 94.6)
- moved C25 182.4 mm to (91.7, 96.6), turned to 180 degrees
- moved U$25 180.4 mm to (110.2, 90.0)
- moved R32 179.9 mm to (66.9, 76.2), flipped to the bottom, turned to 270 degrees
- moved R33 178.8 mm to (68.8, 76.2), flipped to the bottom, turned to 90 degrees
- moved R4 176.1 mm to (124.6, 34.7)
- moved R28 173.9 mm to (36.3, 79.1), flipped to the bottom, turned to 180 degrees
- moved R27 173.7 mm to (36.3, 76.6), flipped to the bottom, turned to 180 degrees
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Connections:
- net USB_DM renamed USB_D_N
- net USB_DP renamed USB_D_PP
- net 3.3V: no longer C19.+
- net GND: now also LED_PWR.C; no longer C19.-, LED3.C
- net N$8: now also LED_PWR.A; no longer LED3.A
Routing:
- net GND: track 12.1 -> 37.1 mm, vias 5 -> 14
- net N$21: track 0.00 -> 15.0 mm
- net N$11: track 0.00 -> 11.6 mm
- net USB_D_PP: track 0.00 -> 9.02 mm
- net USB_D_N: track 0.00 -> 8.89 mm
- net 5.0V: track 0.00 -> 8.39 mm
- net N$10: track 0.00 -> 8.12 mm
- net N$8: track 0.00 -> 1.95 mm
- net 3.3V: track 28.4 -> 30.2 mm

Commit message: wip
Parts:
- C24: value 100nF -> 0.1uF
- moved R14 158.7 mm to (96.3, 72.0)
- moved R11 146.7 mm to (103.3, 72.8), turned to 270 degrees
- moved R12 143.7 mm to (94.0, 70.2)
- moved R10 142.0 mm to (104.9, 72.8), turned to 270 degrees
- moved JTAG 138.2 mm to (85.1, 67.7), turned to 180 degrees
- moved LED2 130.0 mm to (103.3, 76.1)
- moved LED1 127.9 mm to (104.9, 76.1)
- moved R2 127.3 mm to (91.4, 59.7)
- moved R16 115.0 mm to (90.8, 61.8)
- moved R22 105.5 mm to (62.2, 68.7)
- moved R21 98.7 mm to (59.7, 65.5), turned to 270 degrees
- moved R20 98.2 mm to (62.9, 66.4)
- moved C24 74.5 mm to (42.7, 77.3), flipped to the bottom, turned to 90 degrees
- moved H3 65.7 mm to (-8.89, 20.8)
- moved LCD_POT2 50.9 mm to (-8.38, 36.1)
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Connections:
- net SCS_D10: now also R36.1, S3.3, S3.4; no longer SW2.E
- net SCS_D5: now also SW2.E; no longer R36.1, S3.3, S3.4
- net SCS_D6: now also SW2.A; no longer R37.1, S4.3, S4.4
- net SCS_D7: now also SW2.B; no longer R38.1, S5.3, S5.4
- net SCS_D8: now also R38.1, S5.3, S5.4; no longer SW2.B
- net SCS_D9: now also R37.1, S4.3, S4.4; no longer SW2.A
Routing:
- net 5.0V: track 8.39 -> 180.2 mm, vias 0 -> 2
- net SCS_D5: track 0.00 -> 117.4 mm, vias 0 -> 2
- net MIDI_IN1: track 0.00 -> 96.9 mm, vias 0 -> 2
- net MIDI_OUT1: track 0.00 -> 94.0 mm, vias 0 -> 1
- net SCS_D2: track 0.00 -> 91.3 mm
- net SCS_D3: track 0.00 -> 88.5 mm
- net SCS_D4: track 0.00 -> 75.4 mm
- net LCD_RS: track 0.00 -> 67.8 mm, vias 0 -> 3
- net LCD_SER_SCLK: track 0.00 -> 63.6 mm, vias 0 -> 1
- net SCS_D10: track 0.00 -> 62.5 mm
- net LCD_D7: track 0.00 -> 61.4 mm
- net LCD_SER_RCLK: track 0.00 -> 59.5 mm, vias 0 -> 1
- net MIDI_OUT2: track 0.00 -> 57.8 mm, vias 0 -> 1
- net LCD_RW: track 0.00 -> 56.8 mm
- net LCD_E1: track 0.00 -> 54.4 mm, vias 0 -> 3
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
Commit message: wip
Parts:
- removed C11: 0.1uF, microbuilder:0603
- moved R5 157.9 mm to (103.3, 64.4), flipped to the bottom
- moved C18 44.9 mm to (-17.4, 64.1)
- moved H4 44.9 mm to (-10.2, 46.6)
- moved H3 25.8 mm to (-20.3, 43.9)
- moved R8 6.38 mm to (-17.4, 67.8)
- moved R37 4.27 mm to (65.9, 45.1)
- moved R38 3.92 mm to (79.8, 45.1)
- moved R34 1.08 mm to (25.9, 42.8), turned to 180 degrees
- moved FB1 0.76 mm to (103.4, 62.6)
- moved R35 0.74 mm to (39.9, 43.2)
- moved R36 0.28 mm to (53.8, 42.8)
Connections:
- net 3.3V: no longer C11.1
- net GND: no longer C11.2
- net SCS_D0: now also SW2.B; no longer SW1.B
- net SCS_D1: now also SW2.A; no longer SW1.A
- net SCS_D3: now also SW1.B; no longer R34.1, S1.3, S1.4
- net SCS_D4: now also SW1.A; no longer R35.1, S2.3, S2.4
- net SCS_D6: now also R35.1, S2.3, S2.4; no longer SW2.A
- net SCS_D7: now also R34.1, S1.3, S1.4; no longer SW2.B
Routing:
- net SCS_D1: track 0.00 -> 157.3 mm
- net SCS_D0: track 0.00 -> 153.4 mm
- net SCS_D7: track 0.00 -> 134.6 mm, vias 0 -> 2
- net A0: track 8.61 -> 133.6 mm, vias 0 -> 1
- net SCS_D6: track 0.00 -> 121.9 mm, vias 0 -> 2
- net A1: track 8.06 -> 110.2 mm, vias 0 -> 1
- net A2: track 5.69 -> 87.3 mm
- net A3: track 0.00 -> 66.5 mm, vias 0 -> 1
- net SCS_D4: track 75.4 -> 139.7 mm
- net SCS_D2: track 91.3 -> 146.0 mm
- net A4: track 0.00 -> 46.0 mm, vias 0 -> 1
- net SCS_D3: track 88.5 -> 133.3 mm
- net SW_USER: track 6.54 -> 46.1 mm, vias 0 -> 1
- net MIDI_IN1: track 96.9 -> 132.1 mm, vias 2 -> 3
- net MIDI_OUT1: track 94.0 -> 117.8 mm, vias 1 -> 2
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
Commit message: wip
Parts:
- moved SW_USER 139.2 mm to (96.0, 35.2), turned to 270 degrees
- moved SW_RST 134.5 mm to (102.7, 35.2), turned to 90 degrees
- moved R9 133.2 mm to (97.2, 29.1), flipped to the bottom
- moved C18 125.8 mm to (103.4, 28.8), flipped to the bottom, turned to 180 degrees
- moved R8 116.3 mm to (96.0, 41.9), flipped to the bottom, turned to 270 degrees
- moved R15 100.1 mm to (82.3, 65.2), flipped to the bottom, turned to 180 degrees
- moved LCD_POT1 62.5 mm to (34.7, 64.3), turned to 180 degrees
- moved C27 57.6 mm to (94.2, 79.2), flipped to the bottom, turned to 270 degrees
- moved U1 57.2 mm to (86.6, 77.1), flipped to the bottom, turned to 90 degrees
- moved C26 56.5 mm to (94.2, 75.4), flipped to the bottom
- moved R13 53.0 mm to (92.3, 79.1), flipped to the bottom
- moved R17 52.1 mm to (92.3, 75.4), flipped to the bottom, turned to 270 degrees
- moved R4 51.8 mm to (88.4, 71.8), flipped to the bottom
- moved C23 49.6 mm to (88.4, 73.5), flipped to the bottom, turned to 0 degrees
- moved LCD_POT2 43.5 mm to (24.8, 64.3), turned to 180 degrees
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Routing:
- net NRST: track 0.00 -> 71.2 mm, vias 0 -> 1
- net SCL: track 0.00 -> 35.2 mm, vias 0 -> 1
- net SDA: track 0.00 -> 32.4 mm, vias 0 -> 1
- net N$7: track 0.00 -> 16.1 mm, vias 0 -> 2
- net SW_USER: track 46.1 -> 30.7 mm
- net 3.3V: track 31.9 -> 46.1 mm, vias 8 -> 10
- net N$12: track 0.00 -> 12.8 mm
- net MIDI_IN2: track 53.7 -> 49.4 mm
- net N$15: track 5.28 -> 2.66 mm
- net N$17: track 0.00 -> 2.61 mm

Commit message: routed
Parts:
- moved Q1 61.6 mm to (14.1, 67.1)
- moved R19 46.7 mm to (15.0, 62.6)
- moved R18 43.4 mm to (15.0, 64.4)
- moved JP2 39.8 mm to (18.2, 63.4), turned to 270 degrees
- moved C24 1.71 mm to (41.5, 78.6), turned to 180 degrees
Routing:
- net LCD_V0: track 0.00 -> 45.1 mm
- net LCD_VD: track 49.7 -> 87.0 mm
- net LCD_B-: track 0.00 -> 21.6 mm, vias 0 -> 1
- net 5.0V: track 180.2 -> 195.6 mm
- net N$20: track 0.00 -> 14.6 mm
- net N$19: track 0.00 -> 5.02 mm
- net SCS_D7: track 134.6 -> 137.7 mm
- net N$21: track 15.0 -> 17.1 mm
Changed lines of the file:
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@@
 <element name="R17" library="microbuilder" package="0603" value="2.2K" x="92.329" y="75.438" rot="MR270"/>
 <element name="FB1" library="microbuilder" package="_0805" value="" x="103.378" y="62.611" rot="MR180"/>
-<element name="R18" library="microbuilder" package="_0603" value="10K" x="-26.67" y="52.07"/>
-<element name="Q1" library="transistor-small-signal" package="SOT54A" value="BC337" x="-43.18" y="44.45"/>
-<element name="R19" library="microbuilder" package="_0603" value="1K" x="-30.48" y="52.07"/>
-<element name="JP2" library="microbuilder" package="JUMPER3" value="" x="-20.32" y="53.34"/>
+<element name="R18" library="microbuilder" package="_0603" value="10K" x="14.986" y="64.389"/>
+<element name="Q1" library="transistor-small-signal" package="SOT54A" value="BC337" x="14.097" y="67.056"/>
+<element name="R19" library="microbuilder" package="_0603" value="1K" x="14.986" y="62.611"/>
+<element name="JP2" library="microbuilder" package="JUMPER3" value="" x="18.161" y="63.373" rot="R270"/>
 <element name="IC5" library="74xx-eu" package="SO16" value="74HC595D" x="48.895" y="77.597" rot="MR0"/>
-<element name="C24" library="microbuilder" package="0603" value="0.1uF" x="42.672" y="77.343" rot="MR90"/>
+<element name="C24" library="microbuilder" package="0603" value="0.1uF" x="41.529" y="78.613" rot="MR180"/>
 <element name="R20" library="microbuilder" package="_0603" value="1K" x="62.865" y="66.421"/>
 <element name="R21" library="microbuilder" package="_0603" value="1K" x="59.69" y="65.532" rot="R270"/>
@@
 <via x="95.885" y="34.798" extent="1-16" drill="0.3302"/>
 <wire x1="95.885" y1="34.798" x2="96.774" y2="35.687" width="0.254" layer="1"/>
-<wire x1="7.66" y1="20.447" x2="-17.78" y2="53.34" width="0" layer="19" extent="1-1"/>
 </signal>
 <signal name="GND">
@@
 <via x="102.616" y="44.958" extent="1-16" drill="0.3302"/>
 <wire x1="102.616" y1="44.958" x2="102.235" y2="45.339" width="0.254" layer="16"/>
-<wire x1="5.882" y1="59.197" x2="-41.91" y2="44.45" width="0" layer="19" extent="1-1"/>
 </signal>
 <signal name="N$1">
@@
 <wire x1="37.084" y1="81.153" x2="37.084" y2="82.804" width="0.254" layer="1"/>
 <wire x1="37.084" y1="82.804" x2="36.957" y2="82.931" width="0.254" layer="1"/>
-<wire x1="27.311" y1="82.931" x2="27.311" y2="82.81" width="0.254" layer="1"/>
-<wire x1="27.311" y1="82.81" x2="27.305" y2="82.804" width="0.254" layer="1"/>
 <wire x1="18.98" y1="73.33" x2="18.98" y2="73.336" width="0.6096" layer="1"/>
 <wire x1="18.98" y1="73.336" x2="28.575" y2="82.931" width="0.6096" layer="1"/>
@@
 <wire x1="68.326" y1="77.851" x2="57.15" y2="77.851" width="0.254" layer="16"/>
 <wire x1="57.15" y1="77.851" x2="56.896" y2="77.597" width="0.254" layer="16"/>
-<wire x1="28.575" y1="82.931" x2="27.311" y2="82.931" width="0" layer="19" extent="1-1"/>
-<wire x1="22.225" y1="64.262" x2="18.98" y2="73.33" width="0" layer="19" extent="1-1"/>
-<wire x1="-22.86" y1="53.34" x2="18.98" y2="73.33" width="0" layer="19" extent="1-1"/>
-<wire x1="-25.908" y1="52.07" x2="-22.86" y2="53.34" width="0" layer="19" extent="1-1"/>
+<wire x1="18.98" y1="73.33" x2="18.98" y2="66.732" width="0.6096" layer="16"/>
+<wire x1="18.98" y1="66.732" x2="18.161" y2="65.913" width="0.6096" layer="16"/>
+<wire x1="18.161" y1="65.913" x2="20.574" y2="65.913" width="0.4064" layer="16"/>
+<wire x1="20.574" y1="65.913" x2="22.225" y2="64.262" width="0.4064" layer="16"/>
+<wire x1="15.748" y1="64.389" x2="16.637" y2="64.389" width="0.4064" layer="1"/>
+<wire x1="16.637" y1="64.389" x2="18.161" y2="65.913" width="0.4064" layer="1"/>
 </signal>
 <signal name="N$10">
@@
 <contactref element="LCD_POT1" pad="P$2"/>
 <contactref element="LCD1" pad="V5"/>
-<wire x1="34.671" y1="64.262" x2="68.98" y2="71.63" width="0" layer="19" extent="1-1"/>
+<wire x1="68.98" y1="71.63" x2="68.98" y2="62.884" width="0.4064" layer="16"/>
+<wire x1="68.98" y1="62.884" x2="67.183" y2="61.087" width="0.4064" layer="16"/>
+<wire x1="67.183" y1="61.087" x2="37.846" y2="61.087" width="0.4064" layer="16"/>
+<wire x1="37.846" y1="61.087" x2="34.671" y2="64.262" width="0.4064" layer="16"/>
 </signal>
 <signal name="LCD_VD">
@@
 <wire x1="45.72" y1="80.6704" x2="45.72" y2="79.756" width="0.4064" layer="16"/>
 <wire x1="45.72" y1="79.756" x2="44.577" y2="78.613" width="0.4064" layer="16"/>
-<wire x1="44.577" y1="78.613" x2="43.092" y2="78.613" width="0.4064" layer="16"/>
-<wire x1="43.092" y1="78.613" x2="42.672" y2="78.193" width="0.4064" layer="16"/>
+<wire x1="44.577" y1="78.613" x2="42.379" y2="78.613" width="0.4064" layer="16"/>
 <wire x1="58.674" y1="73.406" x2="59.436" y2="73.406" width="0.254" layer="1"/>
 <wire x1="59.436" y1="73.406" x2="59.944" y2="72.898" width="0.254" layer="1"/>
@@
 <wire x1="59.944" y1="70.231" x2="59.944" y2="69.977" width="0.254" layer="1"/>
 <wire x1="59.944" y1="69.977" x2="59.182" y2="69.215" width="0.254" layer="1"/>
-<wire x1="37.211" y1="64.262" x2="42.672" y2="78.193" width="0" layer="19" extent="16-16"/>
-<wire x1="-20.32" y1="53.34" x2="37.211" y2="64.262" width="0" layer="19" extent="1-1"/>
+<wire x1="42.379" y1="78.613" x2="42.379" y2="69.43" width="0.4064" layer="16"/>
+<wire x1="42.379" y1="69.43" x2="37.211" y2="64.262" width="0.4064" layer="16"/>
+<wire x1="18.161" y1="63.373" x2="19.177" y2="63.373" width="0.4064" layer="1"/>
+<wire x1="19.177" y1="63.373" x2="21.59" y2="65.786" width="0.4064" layer="1"/>
+<wire x1="21.59" y1="65.786" x2="35.687" y2="65.786" width="0.4064" layer="1"/>
+<wire x1="35.687" y1="65.786" x2="37.211" y2="64.262" width="0.4064" layer="1"/>
 </signal>
 <signal name="LCD_RS">
@@
 <contactref element="Q1" pad="B"/>
 <contactref element="LCD1" pad="K"/>
-<wire x1="-27.432" y1="52.07" x2="18.98" y2="83.93" width="0" layer="19" extent="1-1"/>
-<wire x1="-43.18" y1="46.355" x2="-27.432" y2="52.07" width="0" layer="19" extent="1-1"/>
+<wire x1="18.98" y1="83.93" x2="18.98" y2="77.654" width="0.4064" layer="1"/>
+<wire x1="18.98" y1="77.654" x2="14.351" y2="73.025" width="0.4064" layer="1"/>
+<via x="14.351" y="73.025" extent="1-16" drill="0.3302"/>
+<wire x1="14.351" y1="73.025" x2="14.351" y2="69.215" width="0.4064" layer="16"/>
+<wire x1="14.351" y1="69.215" x2="14.097" y2="68.961" width="0.4064" layer="16"/>
+<wire x1="14.224" y1="64.389" x2="14.224" y2="68.834" width="0.4064" layer="1"/>
+<wire x1="14.224" y1="68.834" x2="14.097" y2="68.961" width="0.4064" layer="1"/>
 </signal>
 <signal name="LCD_RW">
@@
 <contactref element="R19" pad="1"/>
 <contactref element="Q1" pad="C"/>
-<wire x1="-44.45" y1="44.45" x2="-31.242" y2="52.07" width="0" layer="19" extent="1-1"/>
+<wire x1="12.827" y1="67.056" x2="12.827" y2="64.008" width="0.4064" layer="1"/>
+<wire x1="12.827" y1="64.008" x2="14.224" y2="62.611" width="0.4064" layer="1"/>
 </signal>
 <signal name="N$20">
 <contactref element="R19" pad="2"/>
 <contactref element="LCD_POT2" pad="P$2"/>
-<wire x1="-29.718" y1="52.07" x2="24.765" y2="64.262" width="0" layer="19" extent="1-1"/>
+<wire x1="15.748" y1="62.611" x2="15.748" y2="59.563" width="0.4064" layer="1"/>
+<wire x1="15.748" y1="59.563" x2="16.51" y2="58.801" width="0.4064" layer="1"/>
+<wire x1="16.51" y1="58.801" x2="19.304" y2="58.801" width="0.4064" layer="1"/>
+<wire x1="19.304" y1="58.801" x2="24.765" y2="64.262" width="0.4064" layer="1"/>
 </signal>
 <signal name="LCD_SER_SCLK">
@@
 <wire x1="92.544" y1="91.6296" x2="92.5322" y2="91.6178" width="0.6096" layer="1"/>
 <wire x1="92.5322" y1="91.6178" x2="104.5718" y2="91.6178" width="0.6096" layer="1"/>
-<wire x1="92.544" y1="94.615" x2="92.544" y2="96.647" width="0" layer="19" extent="1-1"/>
+<wire x1="92.544" y1="96.647" x2="92.544" y2="94.615" width="0.6096" layer="1"/>
 </signal>
 <signal name="N$23">
@@
 <wire x1="113.792" y1="66.167" x2="113.538" y2="66.421" width="0.1524" layer="16"/>
 <wire x1="113.792" y1="39.878" x2="113.157" y2="39.243" width="0.1524" layer="16"/>
-<wire x1="26.67" y1="42.799" x2="26.7208" y2="45.9486" width="0" layer="19" extent="1-1"/>
+<wire x1="26.67" y1="42.799" x2="26.67" y2="45.8978" width="0.254" layer="1"/>
+<wire x1="26.67" y1="45.8978" x2="26.7208" y2="45.9486" width="0.254" layer="1"/>
 </signal>
 <signal name="SCS_D8">
@@
 <wire x1="62.484" y1="43.053" x2="62.357" y2="42.926" width="0.1524" layer="1"/>
 <wire x1="97.79" y1="43.18" x2="62.611" y2="43.18" width="0.1524" layer="1"/>
-<wire x1="62.611" y1="43.18" x2="58.928" y2="39.497" width="0.1524" layer="1"/>
+<wire x1="62.357" y1="42.926" x2="58.928" y2="39.497" width="0.1524" layer="1"/>
 <wire x1="58.928" y1="39.497" x2="45.466" y2="39.497" width="0.1524" layer="1"/>
 <wire x1="45.466" y1="39.497" x2="44.831" y2="40.132" width="0.1524" layer="1"/>
@@
 <wire x1="18.923" y1="40.132" x2="10.16" y2="31.369" width="0.1524" layer="16"/>
 <wire x1="10.16" y1="31.369" x2="10.16" y2="20.447" width="0.1524" layer="16"/>
-<wire x1="62.611" y1="43.18" x2="62.484" y2="43.053" width="0" layer="19" extent="1-1"/>
+<wire x1="62.611" y1="43.18" x2="62.484" y2="43.053" width="0.1524" layer="1"/>
 </signal>
 <signal name="A1">

Commit message: all routed
Parts:
- added C3: 0.1uF, microbuilder:0603
- added FLASH1: AT25DF641A or MX25L6406E, vovtech:SOIC-8-WIDE
- added SPI_A: (no value), pinhead:2X06
- added SPI_B: (no value), pinhead:2X07
- moved H3 138.4 mm to (111.8, 2.54)
- moved H4 45.9 mm to (2.54, 2.54)
- moved R2 17.3 mm to (79.1, 47.5)
- moved C8 15.7 mm to (95.1, 41.8), turned to 180 degrees
- moved C4 15.2 mm to (96.5, 43.7), turned to 0 degrees
- moved C5 14.0 mm to (96.4, 45.3), turned to 0 degrees
- moved R16 13.5 mm to (86.2, 49.1)
- moved R1 12.8 mm to (100.5, 46.1)
- moved C13 12.8 mm to (103.9, 46.1)
- moved C15 12.8 mm to (102.2, 46.1)
- moved C12 12.7 mm to (105.8, 46.9)
- moved C14 12.7 mm to (107.4, 46.9)
- moved C7 12.7 mm to (109.2, 46.9)
- moved Y1 12.7 mm to (100.5, 36.4)
- moved R20 12.7 mm to (62.9, 53.7)
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Connections:
- removed net SWO: R16.2, STM32F407XX1.89
- new net A_RC1: SPI_A.12, STM32F407XX1.51
- new net A_RC2: SPI_A.11, STM32F407XX1.57
- new net A_SC: SPI_A.10, SPI_A.9, STM32F407XX1.52
- new net A_SI: SPI_A.7, STM32F407XX1.53
- new net A_SO: SPI_A.8, STM32F407XX1.54
- new net B_RC1: SPI_B.12, STM32F407XX1.77
- new net B_RC2: SPI_B.11, STM32F407XX1.95
- new net B_RC3: SPI_B.14, STM32F407XX1.15
- new net B_RC4: SPI_B.13, STM32F407XX1.18
- new net B_RC5: FLASH1.1, STM32F407XX1.4
- new net B_SC: FLASH1.6, R16.2, SPI_B.10, SPI_B.9, STM32F407XX1.89
- new net B_SI: FLASH1.2, SPI_B.7, STM32F407XX1.90
- new net B_SO: FLASH1.5, SPI_B.8, STM32F407XX1.91
- net 3.3V: now also C3.2, FLASH1.3, FLASH1.7, FLASH1.8, SPI_A.5, SPI_A.6, SPI_B.5, SPI_B.6
- net 5.0V: now also SPI_A.1, SPI_A.2, SPI_B.1, SPI_B.2
- net GND: now also C3.1, FLASH1.4, SPI_A.3, SPI_A.4, SPI_B.3, SPI_B.4
Routing:
- net 5.0V: track 195.6 -> 365.6 mm, vias 2 -> 3
- net A_RC2: track 0.00 -> 79.1 mm, vias 0 -> 3
- net B_SI: track 0.00 -> 76.7 mm, vias 0 -> 2
- net A_SO: track 0.00 -> 75.3 mm, vias 0 -> 2
- net B_SC: track 0.00 -> 74.9 mm, vias 0 -> 1
- net A_SI: track 0.00 -> 73.9 mm, vias 0 -> 2
- net A_SC: track 0.00 -> 71.0 mm, vias 0 -> 1
- net B_RC4: track 0.00 -> 70.2 mm, vias 0 -> 2
- net B_SO: track 0.00 -> 68.8 mm, vias 0 -> 2
- net B_RC3: track 0.00 -> 68.2 mm, vias 0 -> 2
- net B_RC1: track 0.00 -> 67.1 mm, vias 0 -> 3
- net A_RC1: track 0.00 -> 62.9 mm, vias 0 -> 1
- net B_RC5: track 0.00 -> 60.4 mm, vias 0 -> 2
- net B_RC2: track 0.00 -> 57.0 mm, vias 0 -> 3
- net N$5: track 2.15 -> 16.1 mm
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Other:
- board size 114.3 x 101.6 mm -> 114.3 x 88.9 mm
