File: eagle/rev_b/cpu_eval_board.brd (EAGLE design)
At the start: 114.3 x 88.9 mm, 112 parts, among them IC1 6N138S-TA1, IC2 6N138S-TA1, IC5 74HC595D, Q1 BC337, SW1 Encoder, SW2 Encoder, U1 24LC512, Y1 8MHz

Commit message: lcd library edit
Parts:
- moved LCD1 75.3 mm to (23.2, 49.4), turned to 0 degrees
Routing:
- net LCD_RW: track 56.8 -> 75.3 mm
- net LCD_RS: track 67.8 -> 86.1 mm
- net LCD_D6: track 2.90 -> 12.4 mm
- net LCD_D5: track 3.19 -> 12.7 mm
- net LCD_E1: track 53.8 -> 63.2 mm
- net LCD_D4: track 3.49 -> 12.5 mm
- net LCD_D2: track 4.69 -> 13.7 mm
- net LCD_VD: track 87.0 -> 96.0 mm
- net LCD_D3: track 3.80 -> 12.6 mm
- net LCD_D1: track 4.84 -> 13.5 mm
- net LCD_D0: track 12.2 -> 20.4 mm
- net LCD_V0: track 45.1 -> 37.2 mm
- net LCD_B-: track 22.0 -> 19.6 mm
- net LCD_D7: track 61.3 -> 63.1 mm
Changed lines of the file:
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@@
 <attribute name="PARTNO" value="CRCW06031K00FKEA,Vishay / Dale,,71-CRCW0603-1.0K-E3,Thick Film Resistors - SMD 1/10watt 1.0Kohms 1%, REF41" x="68.834" y="63.5" size="1.778" layer="28" rot="MR90" display="off"/>
 </element>
-<element name="LCD1" library="NHD-C0220AA-FSW-FTW" package="NHD-C0220AA-FSW-FTW" value="NHD-C0220AA-FSW-FTW" x="93.98" y="74.93" rot="R180">
-<attribute name="PARTNO" value="NHD-C0220AA-FSW-FTW,Newhaven Display,,763-C0220AA-FSW-FTW,LCD Character Display Modules &amp; Accessories COG FSTN(+) 2x20 White Transflective, REF19" x="93.98" y="74.93" size="1.778" layer="27" rot="R180" display="off"/>
+<element name="LCD1" library="NHD-C0220AA-FSW-FTW" package="NHD-C0220AA-FSW-FTW" value="NHD-C0220AA-FSW-FTW" x="23.1648" y="49.403">
+<attribute name="PARTNO" value="NHD-C0220AA-FSW-FTW,Newhaven Display,,763-C0220AA-FSW-FTW,LCD Character Display Modules &amp; Accessories COG FSTN(+) 2x20 White Transflective, REF19" x="23.1648" y="49.403" size="1.778" layer="27" display="off"/>
 </element>
 <element name="H1" library="holes" package="3,3" value="MOUNT-HOLE3.3" x="2.54" y="86.36"/>
@@
 <wire x1="37.084" y1="68.453" x2="37.084" y2="70.104" width="0.254" layer="1"/>
 <wire x1="37.084" y1="70.104" x2="36.957" y2="70.231" width="0.254" layer="1"/>
-<wire x1="18.98" y1="60.63" x2="18.98" y2="60.636" width="0.6096" layer="1"/>
+<wire x1="18.9148" y1="60.403" x2="18.98" y2="60.636" width="0.6096" layer="1"/>
 <wire x1="18.98" y1="60.636" x2="28.575" y2="70.231" width="0.6096" layer="1"/>
 <wire x1="86.741" y1="72.263" x2="87.376" y2="72.263" width="0.6096" layer="1"/>
@@
 <wire x1="68.326" y1="65.151" x2="57.15" y2="65.151" width="0.254" layer="16"/>
 <wire x1="57.15" y1="65.151" x2="56.896" y2="64.897" width="0.254" layer="16"/>
-<wire x1="18.98" y1="60.63" x2="18.98" y2="54.032" width="0.6096" layer="16"/>
+<wire x1="18.9148" y1="60.403" x2="18.98" y2="54.032" width="0.6096" layer="16"/>
 <wire x1="18.98" y1="54.032" x2="18.161" y2="53.213" width="0.6096" layer="16"/>
 <wire x1="18.161" y1="53.213" x2="20.574" y2="53.213" width="0.4064" layer="16"/>
@@
 <wire x1="9.652" y1="2.54" x2="63.373" y2="2.54" width="0.6096" layer="1"/>
 <wire x1="63.373" y1="2.54" x2="63.754" y2="2.159" width="0.6096" layer="1"/>
-<wire x1="18.929" y1="60.579" x2="18.98" y2="60.63" width="0.6096" layer="1"/>
+<wire x1="18.929" y1="60.579" x2="18.9148" y2="60.403" width="0.6096" layer="1"/>
 <wire x1="2.413" y1="34.417" x2="2.413" y2="9.779" width="0.6096" layer="1"/>
 <wire x1="2.413" y1="9.779" x2="9.652" y2="2.54" width="0.6096" layer="1"/>
@@
 <wire x1="3.302" y1="58.928" x2="6.477" y2="62.103" width="0.6096" layer="16"/>
 <wire x1="6.477" y1="62.103" x2="17.507" y2="62.103" width="0.6096" layer="16"/>
-<wire x1="17.507" y1="62.103" x2="18.98" y2="60.63" width="0.6096" layer="16"/>
+<wire x1="17.507" y1="62.103" x2="18.9148" y2="60.403" width="0.6096" layer="16"/>
 <contactref element="R46" pad="2"/>
 <wire x1="100.33" y1="61.429" x2="100.33" y2="63.5" width="0.1524" layer="1"/>
@@
 <contactref element="LCD1" pad="DB6"/>
 <wire x1="46.99" y1="61.8236" x2="46.99" y2="58.94" width="0.254" layer="16"/>
-<wire x1="46.99" y1="58.94" x2="46.98" y2="58.93" width="0.254" layer="16"/>
+<wire x1="46.99" y1="58.94" x2="46.9148" y2="49.403" width="0.254" layer="16"/>
 </signal>
 <signal name="LCD_D4">
@@
 <contactref element="LCD1" pad="DB4"/>
 <wire x1="49.53" y1="61.8236" x2="49.53" y2="60.38" width="0.1524" layer="16"/>
-<wire x1="49.53" y1="60.38" x2="50.98" y2="58.93" width="0.1524" layer="16"/>
+<wire x1="49.53" y1="60.38" x2="50.9148" y2="49.403" width="0.1524" layer="16"/>
 </signal>
 <signal name="LCD_D2">
@@
 <wire x1="52.07" y1="60.833" x2="52.451" y2="60.452" width="0.1524" layer="16"/>
 <wire x1="52.451" y1="60.452" x2="53.458" y2="60.452" width="0.1524" layer="16"/>
-<wire x1="53.458" y1="60.452" x2="54.98" y2="58.93" width="0.1524" layer="16"/>
+<wire x1="53.458" y1="60.452" x2="54.9148" y2="49.403" width="0.1524" layer="16"/>
 </signal>
 <signal name="LCD_D0">
@@
 <via x="52.451" y="64.897" extent="1-16" drill="0.3302"/>
 <wire x1="52.451" y1="64.897" x2="53.013" y2="64.897" width="0.254" layer="1"/>
-<wire x1="53.013" y1="64.897" x2="58.98" y2="58.93" width="0.254" layer="1"/>
+<wire x1="53.013" y1="64.897" x2="58.9148" y2="49.403" width="0.254" layer="1"/>
 </signal>
 <signal name="LCD_V0">
 <contactref element="LCD_POT1" pad="P$2"/>
 <contactref element="LCD1" pad="V5"/>
-<wire x1="68.98" y1="58.93" x2="68.98" y2="50.184" width="0.4064" layer="16"/>
+<wire x1="68.9148" y1="49.403" x2="68.98" y2="50.184" width="0.4064" layer="16"/>
 <wire x1="68.98" y1="50.184" x2="67.183" y2="48.387" width="0.4064" layer="16"/>
 <wire x1="67.183" y1="48.387" x2="37.846" y2="48.387" width="0.4064" layer="16"/>
@@
 <wire x1="54.61" y1="64.77" x2="58.674" y2="60.706" width="0.4064" layer="1"/>
 <wire x1="58.674" y1="60.706" x2="65.204" y2="60.706" width="0.4064" layer="1"/>
-<wire x1="65.204" y1="60.706" x2="66.98" y2="58.93" width="0.4064" layer="1"/>
+<wire x1="65.204" y1="60.706" x2="66.9148" y2="49.403" width="0.4064" layer="1"/>
 <wire x1="45.72" y1="67.9704" x2="45.72" y2="67.056" width="0.4064" layer="16"/>
 <wire x1="45.72" y1="67.056" x2="44.577" y2="65.913" width="0.4064" layer="16"/>
@@
 <wire x1="65.024" y1="54.61" x2="65.024" y2="58.886" width="0.1524" layer="16"/>
 <wire x1="50.8" y1="67.9704" x2="50.8" y2="64.516" width="0.1524" layer="16"/>
-<wire x1="62.95" y1="60.96" x2="64.98" y2="58.93" width="0.1524" layer="16"/>
+<wire x1="62.95" y1="60.96" x2="64.9148" y2="49.403" width="0.1524" layer="16"/>
 <wire x1="62.95" y1="60.96" x2="56.261" y2="60.96" width="0.1524" layer="16"/>
 <wire x1="53.975" y1="63.881" x2="51.435" y2="63.881" width="0.1524" layer="16"/>
@@
 <wire x1="100.33026875" y1="53.08626875" x2="99.187" y2="51.943" width="0.1524" layer="1"/>
 <wire x1="99.187" y1="51.943" x2="96.393" y2="51.943" width="0.1524" layer="1"/>
-<wire x1="65.024" y1="58.886" x2="64.98" y2="58.93" width="0.1524" layer="16"/>
+<wire x1="65.024" y1="58.886" x2="64.9148" y2="49.403" width="0.1524" layer="16"/>
 </signal>
 <signal name="LCD_D1">
@@
 <contactref element="LCD1" pad="DB1"/>
 <wire x1="53.34" y1="61.8236" x2="54.0864" y2="61.8236" width="0.1524" layer="16"/>
-<wire x1="54.0864" y1="61.8236" x2="56.98" y2="58.93" width="0.1524" layer="16"/>
+<wire x1="54.0864" y1="61.8236" x2="56.9148" y2="49.403" width="0.1524" layer="16"/>
 </signal>
 <signal name="LCD_D3">
@@
 <contactref element="LCD1" pad="DB3"/>
 <wire x1="50.8" y1="61.8236" x2="50.8" y2="61.11" width="0.254" layer="16"/>
-<wire x1="50.8" y1="61.11" x2="52.98" y2="58.93" width="0.1524" layer="16"/>
+<wire x1="50.8" y1="61.11" x2="52.9148" y2="49.403" width="0.1524" layer="16"/>
 </signal>
 <signal name="LCD_D5">
@@
 <wire x1="48.26" y1="60.706" x2="48.895" y2="60.071" width="0.1524" layer="16"/>
 <wire x1="48.895" y1="60.071" x2="48.895" y2="59.015" width="0.1524" layer="16"/>
-<wire x1="48.895" y1="59.015" x2="48.98" y2="58.93" width="0.1524" layer="16"/>
+<wire x1="48.895" y1="59.015" x2="48.9148" y2="49.403" width="0.1524" layer="16"/>
 </signal>
 <signal name="LCD_D7">
@@
 <wire x1="92.948246875" y1="49.672753125" x2="92.583" y2="50.038" width="0.1524" layer="1"/>
 <wire x1="92.583" y1="50.038" x2="45.383" y2="50.038" width="0.1524" layer="1"/>
-<wire x1="44.98" y1="58.93" x2="44.98" y2="50.441" width="0.1524" layer="1"/>
+<wire x1="44.9148" y1="49.403" x2="44.98" y2="50.441" width="0.1524" layer="1"/>
 <wire x1="45.72" y1="61.8236" x2="45.72" y2="59.67" width="0.254" layer="16"/>
-<wire x1="45.72" y1="59.67" x2="44.98" y2="58.93" width="0.254" layer="16"/>
+<wire x1="45.72" y1="59.67" x2="44.9148" y2="49.403" width="0.254" layer="16"/>
 <wire x1="45.383" y1="50.038" x2="44.98" y2="50.441" width="0.1524" layer="1"/>
 </signal>
@@
 <contactref element="Q1" pad="B"/>
 <contactref element="LCD1" pad="K"/>
-<wire x1="18.98" y1="71.23" x2="18.98" y2="64.954" width="0.4064" layer="1"/>
+<wire x1="18.9148" y1="68.903" x2="18.98" y2="64.954" width="0.4064" layer="1"/>
 <wire x1="18.98" y1="64.954" x2="14.351" y2="60.325" width="0.4064" layer="1"/>
 <via x="14.351" y="60.325" extent="1-16" drill="0.3302"/>
@@
 <wire x1="50.165" y1="63.373" x2="53.721" y2="63.373" width="0.1524" layer="16"/>
 <wire x1="56.134" y1="60.452" x2="61.458" y2="60.452" width="0.1524" layer="16"/>
-<wire x1="61.458" y1="60.452" x2="62.98" y2="58.93" width="0.1524" layer="16"/>
+<wire x1="61.458" y1="60.452" x2="62.9148" y2="49.403" width="0.1524" layer="16"/>
 <wire x1="53.975" y1="63.119" x2="53.721" y2="63.373" width="0.1524" layer="16"/>
 <wire x1="56.134" y1="60.452" x2="53.975" y2="62.611" width="0.1524" layer="16"/>
 <wire x1="53.975" y1="62.611" x2="53.975" y2="63.119" width="0.1524" layer="16"/>
 <wire x1="62.992" y1="56.007" x2="62.992" y2="58.918" width="0.1524" layer="1"/>
-<wire x1="62.992" y1="58.918" x2="62.98" y2="58.93" width="0.1524" layer="1"/>
+<wire x1="62.992" y1="58.918" x2="62.9148" y2="49.403" width="0.1524" layer="1"/>
 </signal>
 <signal name="N$19">
@@
 <via x="60.96" y="52.07" extent="1-16" drill="0.3302"/>
 <wire x1="60.96" y1="52.07" x2="60.96" y2="58.91" width="0.254" layer="16"/>
-<wire x1="60.96" y1="58.91" x2="60.98" y2="58.93" width="0.254" layer="16"/>
+<wire x1="60.96" y1="58.91" x2="60.9148" y2="49.403" width="0.254" layer="16"/>
 <wire x1="59.69" y1="52.07" x2="60.96" y2="52.07" width="0.254" layer="1"/>
 <wire x1="101.33026875" y1="57.392753125" x2="101.33026875" y2="53.45126875" width="0.1524" layer="1"/>

Commit message: cpu_eval_board rev b sent to oshpark
Parts:
- moved R35 1.14 mm to (39.9, 29.3)
- moved R38 1.09 mm to (79.1, 31.5)
- moved R37 0.90 mm to (65.8, 31.5)
- moved S1 0.76 mm to (29.2, 38.7)
- moved S2 0.76 mm to (43.2, 38.7)
- moved S3 0.76 mm to (57.1, 38.7)
- moved S4 0.76 mm to (71.1, 38.7)
- moved S5 0.76 mm to (85.1, 38.7)
- moved SW1 0.76 mm to (8.38, 38.7)
- moved R36 0.65 mm to (53.7, 29.5)
- moved R34 0.64 mm to (25.9, 29.5)
Routing:
- net LCD_RW: track 75.3 -> 63.1 mm, vias 0 -> 1
- net LCD_RS: track 86.1 -> 74.0 mm
- net LCD_E1: track 63.2 -> 51.7 mm
- net LCD_VD: track 96.0 -> 85.3 mm
- net LCD_SER_SCLK: track 63.6 -> 68.0 mm
- net N$27: track 17.7 -> 19.1 mm
- net SCS_D5: track 114.1 -> 115.5 mm
- net LCD_D0: track 20.4 -> 21.4 mm, vias 1 -> 2
- net LCD_D7: track 63.1 -> 64.1 mm
- net SCS_D2: track 146.0 -> 145.3 mm
- net SCS_D6: track 126.0 -> 125.3 mm
- net SCS_D7: track 142.9 -> 142.1 mm
- net SCS_D8: track 33.5 -> 34.2 mm
- net LCD_D3: track 12.6 -> 13.3 mm
